Commit message: chang model to sia arm

File: config/robot_6.urdf (robot description, URDF)
Before this commit: robot sia_robot, 8 links, 7 joints
Links:
- removed link link_7
Joints:
- removed joint joint_7
- joint joint_1: origin xyz=0.0 0.0 0.3393 rpy=0 0 0 -> xyz=0.0 0.0 0.1215 rpy=0 0 0
- joint joint_2: origin xyz=0 0 0 rpy=1.5708 0 0 -> xyz=0 -0.1225 0 rpy=1.5708 -1.5708 0
- joint joint_3: origin xyz=0 0.3977 0 rpy=-1.5708 0 0 -> xyz=0.3 0 0 rpy=3.1416 0 0
- joint joint_4: origin xyz=0 0 0 rpy=1.5708 0 0 -> xyz=0.276 0 0.012 rpy=3.1416 0 1.5708
- joint joint_5: origin xyz=0 0.3925 0 rpy=-1.5708 0 0 -> xyz=0 0.09 0 rpy=-1.5708 0 0
- joint joint_6: origin xyz=0 0 0 rpy=1.5708 0 0 -> xyz=0 -0.082 0 rpy=1.5708 0 0
