Commit message: Change To Tech-6

File: config/robot_7.urdf (robot description, URDF)
Before this commit: robot taike_robot, 7 links, 6 joints
Links:
- added link link_7, mass 0.11516; collision mesh filename=package://taike_robot arm_urdf/meshes/link_6.STL; visual mesh filename=package://taike_robot arm_urdf/meshes/link_6.STL
Joints:
- added joint joint_7: type continuous, parent link_6, child link_7, origin xyz=0 0.2145 0 rpy=-1.5708 0 0, axis 0 0 1
- joint joint_1: origin xyz=0.0 0.0 0.1215 rpy=0 0 0 -> xyz=0.0 0.0 0.3393 rpy=0 0 0
- joint joint_2: origin xyz=0 -0.1225 0 rpy=1.5708 -1.5708 0 -> xyz=0 0 0 rpy=1.5708 0 0
- joint joint_3: origin xyz=0.3 0 0 rpy=3.1416 0 0 -> xyz=0 0.3977 0 rpy=-1.5708 0 0
- joint joint_4: origin xyz=0.276 0 0.012 rpy=3.1416 0 1.5708 -> xyz=0 0 0 rpy=1.5708 0 0
- joint joint_5: origin xyz=0 0.09 0 rpy=-1.5708 0 0 -> xyz=0 0.3925 0 rpy=-1.5708 0 0
- joint joint_6: origin xyz=0 -0.082 0 rpy=1.5708 0 0 -> xyz=0 0 0 rpy=1.5708 0 0
