Commit message: update

File: config/robot.urdf (robot description, URDF)
Before this commit: robot taike_robot, 7 links, 6 joints
Links:
- link link_1: mass 1.03091243455262 -> None

Commit message: add parse urdf

File: config/robot.urdf (robot description, URDF)
Before this commit: robot taike_robot, 7 links, 6 joints
Links:
- link base_link: mass 0.47116 -> None

Commit message: test pass :ok:

File: config/robot.urdf (robot description, URDF)
Before this commit: robot taike_robot, 7 links, 6 joints
Joints:
- joint joint_1: origin xyz=-0.00017158 -0.00017422 0.12118 rpy=0 0 0 -> xyz=0.0 0.0 0.1215 rpy=0 0 0
- joint joint_3: axis 0 0 -1 -> 0 0 1; origin xyz=0.3 0 0 rpy=-3.1416 0 0 -> xyz=0.3 0 0 rpy=3.1416 0 0
- joint joint_4: axis 0 0 -1 -> 0 0 1
- joint joint_5: axis 0 0 -1 -> 0 0 1
- joint joint_6: axis 0 0 -1 -> 0 0 1

Commit message: 更新第二款臂的urdf

File: config/robot.urdf (robot description, URDF)
Before this commit: robot sia_robot, 8 links, 7 joints
Joints:
- joint joint_1: origin xyz=0.0 0.0 0.3393 rpy=0 0 0 -> xyz=0.0 0.0 0.34825 rpy=0 0 0
- joint joint_3: origin xyz=0 0.3977 0 rpy=-1.5708 0 0 -> xyz=0 0.41012 0 rpy=-1.5708 0 0
- joint joint_5: origin xyz=0 0.3925 0 rpy=-1.5708 0 0 -> xyz=0 0.40102 0 rpy=-1.5708 0 0
- joint joint_7: origin xyz=0 0.2145 0 rpy=-1.5708 0 0 -> xyz=0 0.22977 0 rpy=-1.5708 0 0

Commit message: 更新第三款机械臂urdf

File: config/robot.urdf (robot description, URDF)
Before this commit: robot sia_robot, 8 links, 7 joints
Joints:
- joint joint_1: origin xyz=0.0 0.0 0.34825 rpy=0 0 0 -> xyz=0.0 0.0 0.3393 rpy=0 0 0
- joint joint_3: origin xyz=0 0.41012 0 rpy=-1.5708 0 0 -> xyz=0 0.3977 0 rpy=-1.5708 0 0
- joint joint_5: origin xyz=0 0.40102 0 rpy=-1.5708 0 0 -> xyz=0 0.3925 0 rpy=-1.5708 0 0
- joint joint_7: origin xyz=0 0.22977 0 rpy=-1.5708 0 0 -> xyz=0 0.2145 0 rpy=-1.5708 0 0

Commit message: 更改URDF的Z轴旋转180

File: config/robot.urdf (robot description, URDF)
Before this commit: robot sia_robot, 8 links, 7 joints
Joints:
- joint joint_2: origin xyz=0 0 0 rpy=1.5708 0 0 -> xyz=0 0 0 rpy=-1.5708 0 0
- joint joint_3: origin xyz=0 0.3977 0 rpy=-1.5708 0 0 -> xyz=0.0  -0.3977  0.0 rpy=1.5708  0.0  0.0
- joint joint_4: origin xyz=0 0 0 rpy=1.5708 0 0 -> xyz=0 0 0 rpy=-1.5708 0 0
- joint joint_5: origin xyz=0 0.3925 0 rpy=-1.5708 0 0 -> xyz=0 -0.3925 0 rpy=1.5708 0 0
- joint joint_6: origin xyz=0 0 0 rpy=1.5708 0 0 -> xyz=0 0 0 rpy=-1.5708 0 0
- joint joint_7: origin xyz=0 0.2145 0 rpy=-1.5708 0 0 -> xyz=0 -0.2145 0 rpy=1.5708 0 0

Commit message: xi-an项目检修

File: config/robot.urdf (robot description, URDF)
Before this commit: robot sia_robot, 8 links, 7 joints
Joints:
- joint joint_1: origin xyz=0.0 0.0 0.3393 rpy=0 0 0 -> xyz=0.0 0.0 0.3393 rpy=0 0 0.37
- joint joint_2: origin xyz=0 0 0 rpy=1.5708 0 0 -> xyz=0 0 0 rpy=-1.5708 0 0
- joint joint_3: origin xyz=0 0.3977 0 rpy=-1.5708 0 0 -> xyz=0.0  -0.3977  0.0 rpy=1.5708  0.0  0.0
- joint joint_4: origin xyz=0 0 0 rpy=1.5708 0 0 -> xyz=0 0 0 rpy=-1.5708 0 0
- joint joint_5: origin xyz=0 0.3925 0 rpy=-1.5708 0 0 -> xyz=0 -0.3925 0 rpy=1.5708 0 0
- joint joint_6: origin xyz=0 0 0 rpy=1.5708 0 0 -> xyz=0 0 0 rpy=-1.5708 0 0
- joint joint_7: origin xyz=0 0.2145 0 rpy=-1.5708 0 0 -> xyz=0 -0.2145 0 rpy=1.5708 0 0

Commit message: 更新urdf为第一台机械臂

File: config/robot.urdf (robot description, URDF)
Before this commit: robot sia_robot, 8 links, 7 joints
Joints:
- joint joint_2: origin xyz=0 0 0 rpy=-1.5708 0 0 -> xyz=0 0 0 rpy=1.5708 0 0
- joint joint_3: origin xyz=0.0  -0.3977  0.0 rpy=1.5708  0.0  0.0 -> xyz=0 0.3977 0 rpy=-1.5708 0 0
- joint joint_4: origin xyz=0 0 0 rpy=-1.5708 0 0 -> xyz=0 0 0 rpy=1.5708 0 0
- joint joint_5: origin xyz=0 -0.3925 0 rpy=1.5708 0 0 -> xyz=0 0.3925 0 rpy=-1.5708 0 0
- joint joint_6: origin xyz=0 0 0 rpy=-1.5708 0 0 -> xyz=0 0 0 rpy=1.5708 0 0
- joint joint_7: origin xyz=0 -0.2145 0 rpy=1.5708 0 0 -> xyz=0 0.2145 0 rpy=-1.5708 0 0

Commit message: 适配车加臂的组合

File: config/robot.urdf (robot description, URDF)
Before this commit: robot sia_robot, 8 links, 7 joints
Links:
- added link link_car, mass 0.11516; collision mesh filename=package://taike_robot arm_urdf/meshes/link_6.STL; visual mesh filename=package://taike_robot arm_urdf/meshes/link_6.STL
- added link link_tip, mass 0.11516; collision mesh filename=package://taike_robot arm_urdf/meshes/link_6.STL; visual mesh filename=package://taike_robot arm_urdf/meshes/link_6.STL
Joints:
- added joint joint_car: type continuous, parent link_7, child link_car, origin xyz=0 0.2145 0 rpy=-1.5708 0 0, axis 0 0 1
- added joint joint_tip: type continuous, parent link_car, child link_tip, origin xyz=0 0.2145 0 rpy=-1.5708 0 0, axis 0 0 1

Commit message: 阻抗控制首次实现

File: config/robot.urdf (robot description, URDF)
Before this commit: robot sia_robot, 8 links, 7 joints
Links:
- removed link link_2
- removed link link_3
- removed link link_4
- removed link link_5
- removed link link_6
- removed link link_7
Joints:
- removed joint joint_2
- removed joint joint_3
- removed joint joint_4
- removed joint joint_5
- removed joint joint_6
- removed joint joint_7
- joint joint_1: origin xyz=0.0 0.0 0.3393 rpy=0 0 0 -> xyz=0.0 0.0 0.1215 rpy=0 0 0

Commit message: 小测最新的ecm和app，测试通过
1.只保留robot.urdf,按照最新的主站字段格式修改urdf，增添type，以及inputs，outputs，
2.本urdf对应科技园7自由度机械臂的eni文件，其他机械臂记得更改关键字段的大小写

File: config/robot.urdf (robot description, URDF)
Before this commit: robot sia_robot, 8 links, 7 joints
Links:
- link link_1: mass None -> 5.683
- link link_2: mass 2.3222 -> 3.99
- link link_3: mass 1.22157164179203 -> 3.685
- link link_4: mass 0.45068 -> 3.185
- link link_5: mass 0.45069 -> 2.932
- link link_6: mass 0.11516 -> 2.043
- link link_7: mass 0.11516 -> 0.994
Joints:
- joint joint_1: origin xyz=0.0 0.0 0.3393 rpy=0 0 0 -> xyz=0.0 0.0 0.348 rpy=0 0 0
- joint joint_3: origin xyz=0 0.3977 0 rpy=-1.5707963267948966 0 0 -> xyz=0 0.41 0 rpy=-1.5707963267948966 0 0
- joint joint_5: origin xyz=0 0.3925 0 rpy=-1.5707963267948966 0 0 -> xyz=0 0.401 0 rpy=-1.5707963267948966 0 0
- joint joint_7: origin xyz=0 0.2145 0 rpy=-1.5707963267948966 0 0 -> xyz=0 0.230 0 rpy=-1.5707963267948966 0 0

Commit message: 添加传感器节点，测试数据读取无误，
1.添加urdf，修改id
2.测试力传感器的数据读取，无误

File: config/robot.urdf (robot description, URDF)
Before this commit: robot sia_robot, 8 links, 7 joints
Links:
- added link link_8, mass 0.994; visual mesh filename=package://self_robot_description/meshes/arm7.STL
Joints:
- added joint joint_8: type fixed, parent link_7, child link_8, origin xyz=0 0.0 0 rpy=0 0 0, axis 0 0 1

Commit message: Fix second arm
1.修改yaml文件路径为etc/rocos-yaml
2. 修改servoj的最大速度柔顺限制

File: config/robot.urdf (robot description, URDF)
Before this commit: robot sia_robot, 9 links, 8 joints
Links:
- removed link link_8
- link link_1: mass 5.683 -> 5.171
- link link_2: mass 3.99 -> 3.958
- link link_3: mass 3.685 -> 3.078
- link link_4: mass 3.185 -> 3.093
- link link_5: mass 2.932 -> 2.549
- link link_6: mass 2.043 -> 2.063
- link link_7: mass 0.994 -> 0.907
Joints:
- removed joint joint_8
- joint joint_1: origin xyz=0.0 0.0 0.348 rpy=0 0 0 -> xyz=0.0 0.0 0.3393 rpy=0 0 0
- joint joint_3: origin xyz=0 0.41 0 rpy=-1.5707963267948966 0 0 -> xyz=0 0.3977 0 rpy=-1.5707963267948966 0 0
- joint joint_5: origin xyz=0 0.401 0 rpy=-1.5707963267948966 0 0 -> xyz=0 0.3925 0 rpy=-1.5707963267948966 0 0
- joint joint_7: origin xyz=0 0.230 0 rpy=-1.5707963267948966 0 0 -> xyz=0 0.2145 0 rpy=-1.5707963267948966 0 0
