Commit message: ①加入SRS构型逆运动求解器 ②替换servoL的迭代法为解析法

File: example/config/robot.urdf (robot description, URDF)
Before this commit: robot sia_robot, 8 links, 7 joints
Links:
- link base_link: geometry collision mesh filename=package://self_robot_description/meshes/base_link.STL; visual mesh filename=package://self_robot_description/meshes/base_link.STL
- link link_1: geometry collision mesh filename=package://self_robot_description/meshes/arm1.STL; visual mesh filename=package://self_robot_description/meshes/arm1.STL
- link link_2: geometry collision mesh filename=package://self_robot_description/meshes/arm2.STL; visual mesh filename=package://self_robot_description/meshes/arm2.STL
- link link_3: geometry collision mesh filename=package://self_robot_description/meshes/arm3.STL; visual mesh filename=package://self_robot_description/meshes/arm3.STL
- link link_4: geometry collision mesh filename=package://self_robot_description/meshes/arm4.STL; visual mesh filename=package://self_robot_description/meshes/arm4.STL
- link link_5: geometry collision mesh filename=package://self_robot_description/meshes/arm5.STL; visual mesh filename=package://self_robot_description/meshes/arm5.STL
- link link_6: geometry collision mesh filename=package://self_robot_description/meshes/arm6.STL; visual mesh filename=package://self_robot_description/meshes/arm6.STL
- link link_7: geometry collision mesh filename=package://self_robot_description/meshes/arm7.STL; visual mesh filename=package://self_robot_description/meshes/arm7.STL
Joints:
- joint joint_2: origin xyz=0 0 0 rpy=1.5708 0 0 -> xyz=0 0 0 rpy=1.5707963267948966 0 0
- joint joint_3: origin xyz=0 0.3977 0 rpy=-1.5708 0 0 -> xyz=0 0.3977 0 rpy=-1.5707963267948966 0 0
- joint joint_4: origin xyz=0 0 0 rpy=1.5708 0 0 -> xyz=0 0 0 rpy=1.5707963267948966 0 0
- joint joint_5: origin xyz=0 0.3925 0 rpy=-1.5708 0 0 -> xyz=0 0.3925 0 rpy=-1.5707963267948966 0 0
- joint joint_6: origin xyz=0 0 0 rpy=1.5708 0 0 -> xyz=0 0 0 rpy=1.5707963267948966 0 0
- joint joint_7: origin xyz=0 0.2145 0 rpy=-1.5708 0 0 -> xyz=0 0.2145 0 rpy=-1.5707963267948966 0 0
