Commit message: update

File: config/models/talon/robot.urdf (robot description, URDF)
Before this commit: robot talon, 8 links, 7 joints
Joints:
- joint joint_5: limit (none) -> lower=-2.71 upper=2.71 effort=30.0

Commit message: update

File: config/models/talon/robot.urdf (robot description, URDF)
Before this commit: robot talon, 8 links, 7 joints
Joints:
- joint joint_5: limit lower=-2.71 upper=2.71 effort=30.0 -> (none)
