Commit message: Add URDF impedance diagnostics and normalize joint torque units
- Add a URDF joint impedance executable with gravity-only compensation testing,
  startup and overspeed snapshots, and aligned theoretical/command torque logs.
- Load rated joint torques from YAML and convert Nm commands and identification
  feedback to and from drive per-mille units.
- Remove the obsolete online single/multi-axis motion implementation and reject
  its HTTP/gRPC motion requests explicitly.
- Include TC7 robot descriptions and meshes with updated joint names, axes,
  hardware mappings and limits.
- Resolve Pinocchio dependencies from ROS 2 Humble and keep HTTP opt-in.

Validation: 100 KDL gravity plus actual-velocity PD reference cases,
bidirectional speed guards, HardwareSim startup/shutdown and log checks.
Python client tests skipped as requested.

File: config/TC7/robot.urdf (robot description, URDF)
Before this commit: robot 7870302-000000-002 TC7-R3B-RevB1-urdf, 8 links, 7 joints
Links:
- link link_7: geometry collision mesh filename=meshes/Link7.STL; visual mesh filename=meshes/Link7.STL
Joints:
- joint joint_1: limit lower=-3.1415 upper=3.1415 effort=10 velocity=2 -> lower=-3.1415 upper=3.1415 effort=100 velocity=2
- joint joint_2: limit lower=-2.3911 upper=2.3911 effort=10 velocity=2 -> lower=-2.3911 upper=2.3911 effort=100 velocity=2
- joint joint_3: limit lower=-3.1415 upper=3.1415 effort=10 velocity=2 -> lower=-3.1415 upper=3.1415 effort=100 velocity=2
- joint joint_4: limit lower=-2.5656 upper=2.5656 effort=10 velocity=2 -> lower=-2.5656 upper=2.5656 effort=100 velocity=2
- joint joint_5: limit lower=-3.1415 upper=3.1415 effort=10 velocity=2 -> lower=-3.1415 upper=3.1415 effort=100 velocity=2
- joint joint_6: limit lower=-2.2166 upper=2.2166 effort=10 velocity=2 -> lower=-2.2166 upper=2.2166 effort=100 velocity=2
- joint joint_7: limit lower=-3.1415 upper=3.1415 effort=10 velocity=2 -> lower=-3.1415 upper=3.1415 effort=100 velocity=2
