Commit message: Update identified impedance models and position-derived velocity feedback
Use measured position differences for excitation recording and identified impedance control. Add configurable friction compensation scaling, updated TC7 identification models, visualization linkage and detailed feedback diagnostics. Preserve exact model URDF bytes for fingerprint validation.

File: config/TC7-robot/TC7-robot.urdf (robot description, URDF)
Before this commit: robot TC7-robot, 8 links, 7 joints
Joints:
- joint joint_1: origin xyz=0 0 0.0823 rpy=0 0 0 -> xyz=0 0 0.0823 rpy=0 0 3.1415926
- joint joint_4: axis 0 0 -1 -> 0 0 1
